File: KiCAD-Rocky-PCB/Rocky-PCB.kicad_pcb (KiCad board)
At the start: 2 copper layers, 122 x 40 mm, 10 parts, among them SW1 PWR SW, U1 ESP32 S3 Sence, U2 BMP390, U3 GY-91, U4 LC76G

Commit message: PCB-V2
Routing:
- net /I2C-SCL: track 176.3 -> 178.3 mm
- net GND: track 182.1 -> 183.3 mm
- net +3.3V: track 115.4 -> 116.6 mm
- net Net-(SW1-B): track 16.2 -> 15.2 mm
